File: left_switches.kicad_sch (KiCad schematic)
At the start: 42 parts, among them SW201 SW_Push, SW202 SW_Push, SW203 SW_Push, SW204 SW_Push, SW205 SW_Push, SW206 SW_Push, SW207 SW_Push, SW208 SW_Push, SW209 SW_Push, SW210 SW_Push, SW211 SW_Push, SW212 SW_Push, SW213 SW_Push, SW214 SW_Push, SW215 SW_Push, SW216 SW_Push, SW217 SW_Push, SW218 SW_Push, SW219 SW_Push, SW220 SW_Push, SW221 SW_Push

Commit message: Make hotswap sockets mountable by JLCPCB
Parts:
- SW201, SW202, SW203, SW204, SW205, SW206, SW207, SW208, SW209, SW210, SW211, SW212, SW213, SW214, SW215, SW216, SW217, SW218, SW219, SW220, SW221: LCSC C2803348 -> C5156480; MFPN PG151101S11 -> CPG151101S11
Changed lines of the file:
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@@
       (effects (font (size 1.27 1.27)) hide)
     )
-    (property "MFPN" "PG151101S11" (at 81.28 72.39 0)
+    (property "MFPN" "CPG151101S11" (at 81.28 72.39 0)
       (effects (font (size 1.27 1.27)) hide)
     )
@@
       (effects (font (size 1.27 1.27)) hide)
     )
-    (property "LCSC" "C2803348" (at 81.28 72.39 0)
+    (property "LCSC" "C5156480" (at 81.28 72.39 0)
       (effects (font (size 1.27 1.27)) hide)
     )
@@
       (effects (font (size 1.27 1.27)) hide)
     )
-    (property "MFPN" "PG151101S11" (at 100.33 59.69 0)
+    (property "MFPN" "CPG151101S11" (at 100.33 59.69 0)
       (effects (font (size 1.27 1.27)) hide)
     )
@@
       (effects (font (size 1.27 1.27)) hide)
     )
-    (property "LCSC" "C2803348" (at 100.33 59.69 0)
+    (property "LCSC" "C5156480" (at 100.33 59.69 0)
       (effects (font (size 1.27 1.27)) hide)
     )
@@
       (effects (font (size 1.27 1.27)) hide)
     )
-    (property "MFPN" "PG151101S11" (at 62.23 59.69 0)
+    (property "MFPN" "CPG151101S11" (at 62.23 59.69 0)
       (effects (font (size 1.27 1.27)) hide)
     )
@@
       (effects (font (size 1.27 1.27)) hide)
     )
-    (property "LCSC" "C2803348" (at 62.23 59.69 0)
+    (property "LCSC" "C5156480" (at 62.23 59.69 0)
       (effects (font (size 1.27 1.27)) hide)
     )
@@
       (effects (font (size 1.27 1.27)) hide)
     )
-    (property "MFPN" "PG151101S11" (at 157.48 46.99 0)
+    (property "MFPN" "CPG151101S11" (at 157.48 46.99 0)
       (effects (font (size 1.27 1.27)) hide)
     )
@@
       (effects (font (size 1.27 1.27)) hide)
     )
-    (property "LCSC" "C2803348" (at 157.48 46.99 0)
+    (property "LCSC" "C5156480" (at 157.48 46.99 0)
       (effects (font (size 1.27 1.27)) hide)
     )
@@
       (effects (font (size 1.27 1.27)) hide)
     )
-    (property "MFPN" "PG151101S11" (at 157.48 59.69 0)
+    (property "MFPN" "CPG151101S11" (at 157.48 59.69 0)
       (effects (font (size 1.27 1.27)) hide)
     )
@@
       (effects (font (size 1.27 1.27)) hide)
     )
-    (property "LCSC" "C2803348" (at 157.48 59.69 0)
+    (property "LCSC" "C5156480" (at 157.48 59.69 0)
       (effects (font (size 1.27 1.27)) hide)
     )
@@
       (effects (font (size 1.27 1.27)) hide)
     )
-    (property "MFPN" "PG151101S11" (at 138.43 46.99 0)
+    (property "MFPN" "CPG151101S11" (at 138.43 46.99 0)
       (effects (font (size 1.27 1.27)) hide)
     )
@@
       (effects (font (size 1.27 1.27)) hide)
     )
-    (property "LCSC" "C2803348" (at 138.43 46.99 0)
+    (property "LCSC" "C5156480" (at 138.43 46.99 0)
       (effects (font (size 1.27 1.27)) hide)
     )
@@
       (effects (font (size 1.27 1.27)) hide)
     )
-    (property "MFPN" "PG151101S11" (at 100.33 72.39 0)
+    (property "MFPN" "CPG151101S11" (at 100.33 72.39 0)
       (effects (font (size 1.27 1.27)) hide)
     )
@@
       (effects (font (size 1.27 1.27)) hide)
     )
-    (property "LCSC" "C2803348" (at 100.33 72.39 0)
+    (property "LCSC" "C5156480" (at 100.33 72.39 0)
       (effects (font (size 1.27 1.27)) hide)
     )
@@
       (effects (font (size 1.27 1.27)) hide)
     )
-    (property "MFPN" "PG151101S11" (at 119.38 72.39 0)
+    (property "MFPN" "CPG151101S11" (at 119.38 72.39 0)
       (effects (font (size 1.27 1.27)) hide)
     )
@@
       (effects (font (size 1.27 1.27)) hide)
     )
-    (property "LCSC" "C2803348" (at 119.38 72.39 0)
+    (property "LCSC" "C5156480" (at 119.38 72.39 0)
       (effects (font (size 1.27 1.27)) hide)
     )
@@
       (effects (font (size 1.27 1.27)) hide)
     )
-    (property "MFPN" "PG151101S11" (at 138.43 85.09 0)
+    (property "MFPN" "CPG151101S11" (at 138.43 85.09 0)
       (effects (font (size 1.27 1.27)) hide)
     )
@@
       (effects (font (size 1.27 1.27)) hide)
     )
-    (property "LCSC" "C2803348" (at 138.43 85.09 0)
+    (property "LCSC" "C5156480" (at 138.43 85.09 0)
       (effects (font (size 1.27 1.27)) hide)
     )
@@
       (effects (font (size 1.27 1.27)) hide)
     )
-    (property "MFPN" "PG151101S11" (at 138.43 72.39 0)
+    (property "MFPN" "CPG151101S11" (at 138.43 72.39 0)
       (effects (font (size 1.27 1.27)) hide)
     )
@@
       (effects (font (size 1.27 1.27)) hide)
     )
-    (property "LCSC" "C2803348" (at 138.43 72.39 0)
+    (property "LCSC" "C5156480" (at 138.43 72.39 0)
       (effects (font (size 1.27 1.27)) hide)
     )
@@
       (effects (font (size 1.27 1.27)) hide)
     )
-    (property "MFPN" "PG151101S11" (at 62.23 72.39 0)
+    (property "MFPN" "CPG151101S11" (at 62.23 72.39 0)
       (effects (font (size 1.27 1.27)) hide)
     )
@@
       (effects (font (size 1.27 1.27)) hide)
     )
-    (property "LCSC" "C2803348" (at 62.23 72.39 0)
+    (property "LCSC" "C5156480" (at 62.23 72.39 0)
       (effects (font (size 1.27 1.27)) hide)
     )
@@
       (effects (font (size 1.27 1.27)) hide)
     )
-    (property "MFPN" "PG151101S11" (at 157.48 85.09 0)
+    (property "MFPN" "CPG151101S11" (at 157.48 85.09 0)
       (effects (font (size 1.27 1.27)) hide)
     )
@@
       (effects (font (size 1.27 1.27)) hide)
     )
-    (property "LCSC" "C2803348" (at 157.48 85.09 0)
+    (property "LCSC" "C5156480" (at 157.48 85.09 0)
       (effects (font (size 1.27 1.27)) hide)
     )
@@
       (effects (font (size 1.27 1.27)) hide)
     )
-    (property "MFPN" "PG151101S11" (at 119.38 59.69 0)
+    (property "MFPN" "CPG151101S11" (at 119.38 59.69 0)
       (effects (font (size 1.27 1.27)) hide)
     )
@@
       (effects (font (size 1.27 1.27)) hide)
     )
-    (property "LCSC" "C2803348" (at 119.38 59.69 0)
+    (property "LCSC" "C5156480" (at 119.38 59.69 0)
       (effects (font (size 1.27 1.27)) hide)
     )
@@
       (effects (font (size 1.27 1.27)) hide)
     )
-    (property "MFPN" "PG151101S11" (at 81.28 59.69 0)
+    (property "MFPN" "CPG151101S11" (at 81.28 59.69 0)
       (effects (font (size 1.27 1.27)) hide)
     )
@@
       (effects (font (size 1.27 1.27)) hide)
     )
-    (property "LCSC" "C2803348" (at 81.28 59.69 0)
+    (property "LCSC" "C5156480" (at 81.28 59.69 0)
       (effects (font (size 1.27 1.27)) hide)
     )
@@
       (effects (font (size 1.27 1.27)) hide)
     )
-    (property "MFPN" "PG151101S11" (at 119.38 46.99 0)
+    (property "MFPN" "CPG151101S11" (at 119.38 46.99 0)
       (effects (font (size 1.27 1.27)) hide)
     )
@@
       (effects (font (size 1.27 1.27)) hide)
     )
-    (property "LCSC" "C2803348" (at 119.38 46.99 0)
+    (property "LCSC" "C5156480" (at 119.38 46.99 0)
       (effects (font (size 1.27 1.27)) hide)
     )
@@
       (effects (font (size 1.27 1.27)) hide)
     )
-    (property "MFPN" "PG151101S11" (at 119.38 85.09 0)
+    (property "MFPN" "CPG151101S11" (at 119.38 85.09 0)
       (effects (font (size 1.27 1.27)) hide)
     )
@@
       (effects (font (size 1.27 1.27)) hide)
     )
-    (property "LCSC" "C2803348" (at 119.38 85.09 0)
+    (property "LCSC" "C5156480" (at 119.38 85.09 0)
       (effects (font (size 1.27 1.27)) hide)
     )
@@
       (effects (font (size 1.27 1.27)) hide)
     )
-    (property "MFPN" "PG151101S11" (at 81.28 46.99 0)
+    (property "MFPN" "CPG151101S11" (at 81.28 46.99 0)
       (effects (font (size 1.27 1.27)) hide)
     )
@@
       (effects (font (size 1.27 1.27)) hide)
     )
-    (property "LCSC" "C2803348" (at 81.28 46.99 0)
+    (property "LCSC" "C5156480" (at 81.28 46.99 0)
       (effects (font (size 1.27 1.27)) hide)
     )
@@
       (effects (font (size 1.27 1.27)) hide)
     )
-    (property "MFPN" "PG151101S11" (at 62.23 46.99 0)
+    (property "MFPN" "CPG151101S11" (at 62.23 46.99 0)
       (effects (font (size 1.27 1.27)) hide)
     )
@@
       (effects (font (size 1.27 1.27)) hide)
     )
-    (property "LCSC" "C2803348" (at 62.23 46.99 0)
+    (property "LCSC" "C5156480" (at 62.23 46.99 0)
       (effects (font (size 1.27 1.27)) hide)
     )
@@
       (effects (font (size 1.27 1.27)) hide)
     )
-    (property "MFPN" "PG151101S11" (at 138.43 59.69 0)
+    (property "MFPN" "CPG151101S11" (at 138.43 59.69 0)
       (effects (font (size 1.27 1.27)) hide)
     )
@@
       (effects (font (size 1.27 1.27)) hide)
     )
-    (property "LCSC" "C2803348" (at 138.43 59.69 0)
+    (property "LCSC" "C5156480" (at 138.43 59.69 0)
       (effects (font (size 1.27 1.27)) hide)
     )
@@
       (effects (font (size 1.27 1.27)) hide)
     )
-    (property "MFPN" "PG151101S11" (at 157.48 72.39 0)
+    (property "MFPN" "CPG151101S11" (at 157.48 72.39 0)
       (effects (font (size 1.27 1.27)) hide)
     )
@@
       (effects (font (size 1.27 1.27)) hide)
     )
-    (property "LCSC" "C2803348" (at 157.48 72.39 0)
+    (property "LCSC" "C5156480" (at 157.48 72.39 0)
       (effects (font (size 1.27 1.27)) hide)
     )
@@
       (effects (font (size 1.27 1.27)) hide)
     )
-    (property "MFPN" "PG151101S11" (at 100.33 46.99 0)
+    (property "MFPN" "CPG151101S11" (at 100.33 46.99 0)
       (effects (font (size 1.27 1.27)) hide)
     )
@@
       (effects (font (size 1.27 1.27)) hide)
     )
-    (property "LCSC" "C2803348" (at 100.33 46.99 0)
-      (effects (font (size 1.27 1.27)) hide)
-    )
+    (property "LCSC" "C5156480" (at 100.33 46.99 0)
+      (effects (font (size 1.27 1.27)) hide)
+    )
