File: right_switches.kicad_sch (KiCad schematic)
At the start: 42 parts, among them SW201 SW_Push, SW202 SW_Push, SW203 SW_Push, SW204 SW_Push, SW205 SW_Push, SW206 SW_Push, SW207 SW_Push, SW208 SW_Push, SW209 SW_Push, SW210 SW_Push, SW211 SW_Push, SW212 SW_Push, SW213 SW_Push, SW214 SW_Push, SW215 SW_Push, SW216 SW_Push, SW217 SW_Push, SW218 SW_Push, SW219 SW_Push, SW220 SW_Push, SW221 SW_Push

Commit message: Make hotswap sockets mountable by JLCPCB
Parts:
- SW201, SW202, SW203, SW204, SW205, SW206, SW207, SW208, SW209, SW210, SW211, SW212, SW213, SW214, SW215, SW216, SW217, SW218, SW219, SW220, SW221: LCSC C2803348 -> C5156480; MFPN PG151101S11 -> CPG151101S11
Changed lines of the file:
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@@
       (effects (font (size 1.27 1.27)) hide)
     )
-    (property "MFPN" "PG151101S11" (at 119.38 72.39 0)
+    (property "MFPN" "CPG151101S11" (at 119.38 72.39 0)
       (effects (font (size 1.27 1.27)) hide)
     )
@@
       (effects (font (size 1.27 1.27)) hide)
     )
-    (property "LCSC" "C2803348" (at 119.38 72.39 0)
+    (property "LCSC" "C5156480" (at 119.38 72.39 0)
       (effects (font (size 1.27 1.27)) hide)
     )
@@
       (effects (font (size 1.27 1.27)) hide)
     )
-    (property "MFPN" "PG151101S11" (at 100.33 59.69 0)
+    (property "MFPN" "CPG151101S11" (at 100.33 59.69 0)
       (effects (font (size 1.27 1.27)) hide)
     )
@@
       (effects (font (size 1.27 1.27)) hide)
     )
-    (property "LCSC" "C2803348" (at 100.33 59.69 0)
+    (property "LCSC" "C5156480" (at 100.33 59.69 0)
       (effects (font (size 1.27 1.27)) hide)
     )
@@
       (effects (font (size 1.27 1.27)) hide)
     )
-    (property "MFPN" "PG151101S11" (at 138.43 72.39 0)
+    (property "MFPN" "CPG151101S11" (at 138.43 72.39 0)
       (effects (font (size 1.27 1.27)) hide)
     )
@@
       (effects (font (size 1.27 1.27)) hide)
     )
-    (property "LCSC" "C2803348" (at 138.43 72.39 0)
+    (property "LCSC" "C5156480" (at 138.43 72.39 0)
       (effects (font (size 1.27 1.27)) hide)
     )
@@
       (effects (font (size 1.27 1.27)) hide)
     )
-    (property "MFPN" "PG151101S11" (at 81.28 72.39 0)
+    (property "MFPN" "CPG151101S11" (at 81.28 72.39 0)
       (effects (font (size 1.27 1.27)) hide)
     )
@@
       (effects (font (size 1.27 1.27)) hide)
     )
-    (property "LCSC" "C2803348" (at 81.28 72.39 0)
+    (property "LCSC" "C5156480" (at 81.28 72.39 0)
       (effects (font (size 1.27 1.27)) hide)
     )
@@
       (effects (font (size 1.27 1.27)) hide)
     )
-    (property "MFPN" "PG151101S11" (at 100.33 72.39 0)
+    (property "MFPN" "CPG151101S11" (at 100.33 72.39 0)
       (effects (font (size 1.27 1.27)) hide)
     )
@@
       (effects (font (size 1.27 1.27)) hide)
     )
-    (property "LCSC" "C2803348" (at 100.33 72.39 0)
+    (property "LCSC" "C5156480" (at 100.33 72.39 0)
       (effects (font (size 1.27 1.27)) hide)
     )
@@
       (effects (font (size 1.27 1.27)) hide)
     )
-    (property "MFPN" "PG151101S11" (at 119.38 46.99 0)
+    (property "MFPN" "CPG151101S11" (at 119.38 46.99 0)
       (effects (font (size 1.27 1.27)) hide)
     )
@@
       (effects (font (size 1.27 1.27)) hide)
     )
-    (property "LCSC" "C2803348" (at 119.38 46.99 0)
+    (property "LCSC" "C5156480" (at 119.38 46.99 0)
       (effects (font (size 1.27 1.27)) hide)
     )
@@
       (effects (font (size 1.27 1.27)) hide)
     )
-    (property "MFPN" "PG151101S11" (at 100.33 46.99 0)
+    (property "MFPN" "CPG151101S11" (at 100.33 46.99 0)
       (effects (font (size 1.27 1.27)) hide)
     )
@@
       (effects (font (size 1.27 1.27)) hide)
     )
-    (property "LCSC" "C2803348" (at 100.33 46.99 0)
+    (property "LCSC" "C5156480" (at 100.33 46.99 0)
       (effects (font (size 1.27 1.27)) hide)
     )
@@
       (effects (font (size 1.27 1.27)) hide)
     )
-    (property "MFPN" "PG151101S11" (at 138.43 46.99 0)
+    (property "MFPN" "CPG151101S11" (at 138.43 46.99 0)
       (effects (font (size 1.27 1.27)) hide)
     )
@@
       (effects (font (size 1.27 1.27)) hide)
     )
-    (property "LCSC" "C2803348" (at 138.43 46.99 0)
+    (property "LCSC" "C5156480" (at 138.43 46.99 0)
       (effects (font (size 1.27 1.27)) hide)
     )
@@
       (effects (font (size 1.27 1.27)) hide)
     )
-    (property "MFPN" "PG151101S11" (at 157.48 85.09 0)
+    (property "MFPN" "CPG151101S11" (at 157.48 85.09 0)
       (effects (font (size 1.27 1.27)) hide)
     )
@@
       (effects (font (size 1.27 1.27)) hide)
     )
-    (property "LCSC" "C2803348" (at 157.48 85.09 0)
+    (property "LCSC" "C5156480" (at 157.48 85.09 0)
       (effects (font (size 1.27 1.27)) hide)
     )
@@
       (effects (font (size 1.27 1.27)) hide)
     )
-    (property "MFPN" "PG151101S11" (at 62.23 46.99 0)
+    (property "MFPN" "CPG151101S11" (at 62.23 46.99 0)
       (effects (font (size 1.27 1.27)) hide)
     )
@@
       (effects (font (size 1.27 1.27)) hide)
     )
-    (property "LCSC" "C2803348" (at 62.23 46.99 0)
+    (property "LCSC" "C5156480" (at 62.23 46.99 0)
       (effects (font (size 1.27 1.27)) hide)
     )
@@
       (effects (font (size 1.27 1.27)) hide)
     )
-    (property "MFPN" "PG151101S11" (at 62.23 72.39 0)
+    (property "MFPN" "CPG151101S11" (at 62.23 72.39 0)
       (effects (font (size 1.27 1.27)) hide)
     )
@@
       (effects (font (size 1.27 1.27)) hide)
     )
-    (property "LCSC" "C2803348" (at 62.23 72.39 0)
+    (property "LCSC" "C5156480" (at 62.23 72.39 0)
       (effects (font (size 1.27 1.27)) hide)
     )
@@
       (effects (font (size 1.27 1.27)) hide)
     )
-    (property "MFPN" "PG151101S11" (at 157.48 46.99 0)
+    (property "MFPN" "CPG151101S11" (at 157.48 46.99 0)
       (effects (font (size 1.27 1.27)) hide)
     )
@@
       (effects (font (size 1.27 1.27)) hide)
     )
-    (property "LCSC" "C2803348" (at 157.48 46.99 0)
+    (property "LCSC" "C5156480" (at 157.48 46.99 0)
       (effects (font (size 1.27 1.27)) hide)
     )
@@
       (effects (font (size 1.27 1.27)) hide)
     )
-    (property "MFPN" "PG151101S11" (at 119.38 59.69 0)
+    (property "MFPN" "CPG151101S11" (at 119.38 59.69 0)
       (effects (font (size 1.27 1.27)) hide)
     )
@@
       (effects (font (size 1.27 1.27)) hide)
     )
-    (property "LCSC" "C2803348" (at 119.38 59.69 0)
+    (property "LCSC" "C5156480" (at 119.38 59.69 0)
       (effects (font (size 1.27 1.27)) hide)
     )
@@
       (effects (font (size 1.27 1.27)) hide)
     )
-    (property "MFPN" "PG151101S11" (at 119.38 85.09 0)
+    (property "MFPN" "CPG151101S11" (at 119.38 85.09 0)
       (effects (font (size 1.27 1.27)) hide)
     )
@@
       (effects (font (size 1.27 1.27)) hide)
     )
-    (property "LCSC" "C2803348" (at 119.38 85.09 0)
+    (property "LCSC" "C5156480" (at 119.38 85.09 0)
       (effects (font (size 1.27 1.27)) hide)
     )
@@
       (effects (font (size 1.27 1.27)) hide)
     )
-    (property "MFPN" "PG151101S11" (at 81.28 59.69 0)
+    (property "MFPN" "CPG151101S11" (at 81.28 59.69 0)
       (effects (font (size 1.27 1.27)) hide)
     )
@@
       (effects (font (size 1.27 1.27)) hide)
     )
-    (property "LCSC" "C2803348" (at 81.28 59.69 0)
+    (property "LCSC" "C5156480" (at 81.28 59.69 0)
       (effects (font (size 1.27 1.27)) hide)
     )
@@
       (effects (font (size 1.27 1.27)) hide)
     )
-    (property "MFPN" "PG151101S11" (at 157.48 59.69 0)
+    (property "MFPN" "CPG151101S11" (at 157.48 59.69 0)
       (effects (font (size 1.27 1.27)) hide)
     )
@@
       (effects (font (size 1.27 1.27)) hide)
     )
-    (property "LCSC" "C2803348" (at 157.48 59.69 0)
+    (property "LCSC" "C5156480" (at 157.48 59.69 0)
       (effects (font (size 1.27 1.27)) hide)
     )
@@
       (effects (font (size 1.27 1.27)) hide)
     )
-    (property "MFPN" "PG151101S11" (at 138.43 85.09 0)
+    (property "MFPN" "CPG151101S11" (at 138.43 85.09 0)
       (effects (font (size 1.27 1.27)) hide)
     )
@@
       (effects (font (size 1.27 1.27)) hide)
     )
-    (property "LCSC" "C2803348" (at 138.43 85.09 0)
+    (property "LCSC" "C5156480" (at 138.43 85.09 0)
       (effects (font (size 1.27 1.27)) hide)
     )
@@
       (effects (font (size 1.27 1.27)) hide)
     )
-    (property "MFPN" "PG151101S11" (at 62.23 59.69 0)
+    (property "MFPN" "CPG151101S11" (at 62.23 59.69 0)
       (effects (font (size 1.27 1.27)) hide)
     )
@@
       (effects (font (size 1.27 1.27)) hide)
     )
-    (property "LCSC" "C2803348" (at 62.23 59.69 0)
+    (property "LCSC" "C5156480" (at 62.23 59.69 0)
       (effects (font (size 1.27 1.27)) hide)
     )
@@
       (effects (font (size 1.27 1.27)) hide)
     )
-    (property "MFPN" "PG151101S11" (at 138.43 59.69 0)
+    (property "MFPN" "CPG151101S11" (at 138.43 59.69 0)
       (effects (font (size 1.27 1.27)) hide)
     )
@@
       (effects (font (size 1.27 1.27)) hide)
     )
-    (property "LCSC" "C2803348" (at 138.43 59.69 0)
+    (property "LCSC" "C5156480" (at 138.43 59.69 0)
       (effects (font (size 1.27 1.27)) hide)
     )
@@
       (effects (font (size 1.27 1.27)) hide)
     )
-    (property "MFPN" "PG151101S11" (at 81.28 46.99 0)
+    (property "MFPN" "CPG151101S11" (at 81.28 46.99 0)
       (effects (font (size 1.27 1.27)) hide)
     )
@@
       (effects (font (size 1.27 1.27)) hide)
     )
-    (property "LCSC" "C2803348" (at 81.28 46.99 0)
+    (property "LCSC" "C5156480" (at 81.28 46.99 0)
       (effects (font (size 1.27 1.27)) hide)
     )
@@
       (effects (font (size 1.27 1.27)) hide)
     )
-    (property "MFPN" "PG151101S11" (at 157.48 72.39 0)
+    (property "MFPN" "CPG151101S11" (at 157.48 72.39 0)
       (effects (font (size 1.27 1.27)) hide)
     )
@@
       (effects (font (size 1.27 1.27)) hide)
     )
-    (property "LCSC" "C2803348" (at 157.48 72.39 0)
-      (effects (font (size 1.27 1.27)) hide)
-    )
+    (property "LCSC" "C5156480" (at 157.48 72.39 0)
+      (effects (font (size 1.27 1.27)) hide)
+    )

Commit message: Save
Connections:
- net COL0: now also SW201.1, SW207.1, SW213.1; no longer SW201.2, SW207.2, SW213.2
- net COL1: now also SW202.1, SW208.1, SW214.1; no longer SW202.2, SW208.2, SW214.2
- net COL2: now also SW203.1, SW209.1, SW215.1; no longer SW203.2, SW209.2, SW215.2
- net COL3: now also SW204.1, SW210.1, SW216.1; no longer SW204.2, SW210.2, SW216.2
- net COL4: now also SW205.1, SW211.1, SW217.1; no longer SW205.2, SW211.2, SW217.2
- net COL5: now also SW206.1, SW212.1, SW218.1; no longer SW206.2, SW212.2, SW218.2
- net at D216.2 (A): now also SW216.2; no longer SW216.1
- net at D201.2 (A): now also SW201.2; no longer SW201.1
- net at D211.2 (A): now also SW211.2; no longer SW211.1
- net at D203.2 (A): now also SW203.2; no longer SW203.1
- net at D209.2 (A): now also SW209.2; no longer SW209.1
- net at D217.2 (A): now also SW217.2; no longer SW217.1
- net at D214.2 (A): now also SW214.2; no longer SW214.1
- net at D215.2 (A): now also SW215.2; no longer SW215.1
- net at D204.2 (A): now also SW204.2; no longer SW204.1
- net at D205.2 (A): now also SW205.2; no longer SW205.1
- net at D213.2 (A): now also SW213.2; no longer SW213.1
- net at D218.2 (A): now also SW218.2; no longer SW218.1
- net at D206.2 (A): now also SW206.2; no longer SW206.1
- net at D210.2 (A): now also SW210.2; no longer SW210.1
- net at D208.2 (A): now also SW208.2; no longer SW208.1
- net at D212.2 (A): now also SW212.2; no longer SW212.1
- net at D207.2 (A): now also SW207.2; no longer SW207.1
- net at D202.2 (A): now also SW202.2; no longer SW202.1
Changed lines of the file:
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@@
     (effects (font (size 1.27 1.27)) (justify left))
   )
-  (symbol (lib_id "Switch:SW_Push") (at 119.38 72.39 0) (mirror y) (unit 1)
+  (symbol (lib_id "Switch:SW_Push") (at 119.38 72.39 0) (unit 1)
     (in_bom yes) (on_board yes) (dnp no)
     (property "Reference" "SW216" (at 119.38 67.31 0)
@@
     )
   )
-  (symbol (lib_id "Switch:SW_Push") (at 100.33 59.69 0) (mirror y) (unit 1)
+  (symbol (lib_id "Switch:SW_Push") (at 100.33 59.69 0) (unit 1)
     (in_bom yes) (on_board yes) (dnp no)
     (property "Reference" "SW209" (at 100.33 54.61 0)
@@
     )
   )
-  (symbol (lib_id "Switch:SW_Push") (at 138.43 72.39 0) (mirror y) (unit 1)
+  (symbol (lib_id "Switch:SW_Push") (at 138.43 72.39 0) (unit 1)
     (in_bom yes) (on_board yes) (dnp no)
     (property "Reference" "SW217" (at 138.43 67.31 0)
@@
     )
   )
-  (symbol (lib_id "Switch:SW_Push") (at 81.28 72.39 0) (mirror y) (unit 1)
+  (symbol (lib_id "Switch:SW_Push") (at 81.28 72.39 0) (unit 1)
     (in_bom yes) (on_board yes) (dnp no)
     (property "Reference" "SW214" (at 81.28 67.31 0)
@@
     )
   )
-  (symbol (lib_id "Switch:SW_Push") (at 100.33 72.39 0) (mirror y) (unit 1)
+  (symbol (lib_id "Switch:SW_Push") (at 100.33 72.39 0) (unit 1)
     (in_bom yes) (on_board yes) (dnp no)
     (property "Reference" "SW215" (at 100.33 67.31 0)
@@
     )
   )
-  (symbol (lib_id "Switch:SW_Push") (at 119.38 46.99 0) (mirror y) (unit 1)
+  (symbol (lib_id "Switch:SW_Push") (at 119.38 46.99 0) (unit 1)
     (in_bom yes) (on_board yes) (dnp no)
     (property "Reference" "SW204" (at 119.38 41.91 0)
@@
     )
   )
-  (symbol (lib_id "Switch:SW_Push") (at 100.33 46.99 0) (mirror y) (unit 1)
+  (symbol (lib_id "Switch:SW_Push") (at 100.33 46.99 0) (unit 1)
     (in_bom yes) (on_board yes) (dnp no)
     (property "Reference" "SW203" (at 100.33 41.91 0)
@@
     )
   )
-  (symbol (lib_id "Switch:SW_Push") (at 138.43 46.99 0) (mirror y) (unit 1)
+  (symbol (lib_id "Switch:SW_Push") (at 138.43 46.99 0) (unit 1)
     (in_bom yes) (on_board yes) (dnp no)
     (property "Reference" "SW205" (at 138.43 41.91 0)
@@
     )
   )
-  (symbol (lib_id "Switch:SW_Push") (at 62.23 46.99 0) (mirror y) (unit 1)
+  (symbol (lib_id "Switch:SW_Push") (at 62.23 46.99 0) (unit 1)
     (in_bom yes) (on_board yes) (dnp no)
     (property "Reference" "SW201" (at 62.23 41.91 0)
@@
     )
   )
-  (symbol (lib_id "Switch:SW_Push") (at 62.23 72.39 0) (mirror y) (unit 1)
+  (symbol (lib_id "Switch:SW_Push") (at 62.23 72.39 0) (unit 1)
     (in_bom yes) (on_board yes) (dnp no)
     (property "Reference" "SW213" (at 62.23 67.31 0)
@@
     )
   )
-  (symbol (lib_id "Switch:SW_Push") (at 157.48 46.99 0) (mirror y) (unit 1)
+  (symbol (lib_id "Switch:SW_Push") (at 157.48 46.99 0) (unit 1)
     (in_bom yes) (on_board yes) (dnp no)
     (property "Reference" "SW206" (at 157.48 41.91 0)
@@
     )
   )
-  (symbol (lib_id "Switch:SW_Push") (at 119.38 59.69 0) (mirror y) (unit 1)
+  (symbol (lib_id "Switch:SW_Push") (at 119.38 59.69 0) (unit 1)
     (in_bom yes) (on_board yes) (dnp no)
     (property "Reference" "SW210" (at 119.38 54.61 0)
@@
     )
   )
-  (symbol (lib_id "Switch:SW_Push") (at 81.28 59.69 0) (mirror y) (unit 1)
+  (symbol (lib_id "Switch:SW_Push") (at 81.28 59.69 0) (unit 1)
     (in_bom yes) (on_board yes) (dnp no)
     (property "Reference" "SW208" (at 81.28 54.61 0)
@@
     )
   )
-  (symbol (lib_id "Switch:SW_Push") (at 157.48 59.69 0) (mirror y) (unit 1)
+  (symbol (lib_id "Switch:SW_Push") (at 157.48 59.69 0) (unit 1)
     (in_bom yes) (on_board yes) (dnp no)
     (property "Reference" "SW212" (at 157.48 54.61 0)
@@
     )
   )
-  (symbol (lib_id "Switch:SW_Push") (at 62.23 59.69 0) (mirror y) (unit 1)
+  (symbol (lib_id "Switch:SW_Push") (at 62.23 59.69 0) (unit 1)
     (in_bom yes) (on_board yes) (dnp no)
     (property "Reference" "SW207" (at 62.23 54.61 0)
@@
     )
   )
-  (symbol (lib_id "Switch:SW_Push") (at 138.43 59.69 0) (mirror y) (unit 1)
+  (symbol (lib_id "Switch:SW_Push") (at 138.43 59.69 0) (unit 1)
     (in_bom yes) (on_board yes) (dnp no)
     (property "Reference" "SW211" (at 138.43 54.61 0)
@@
     )
   )
-  (symbol (lib_id "Switch:SW_Push") (at 81.28 46.99 0) (mirror y) (unit 1)
+  (symbol (lib_id "Switch:SW_Push") (at 81.28 46.99 0) (unit 1)
     (in_bom yes) (on_board yes) (dnp no)
     (property "Reference" "SW202" (at 81.28 41.91 0)
@@
     )
   )
-  (symbol (lib_id "Switch:SW_Push") (at 157.48 72.39 0) (mirror y) (unit 1)
+  (symbol (lib_id "Switch:SW_Push") (at 157.48 72.39 0) (unit 1)
     (in_bom yes) (on_board yes) (dnp no)
     (property "Reference" "SW218" (at 157.48 67.31 0)
