File: crkbd-shockburst.kicad_pcb (KiCad board)
At the start: 4 copper layers, 272 x 112 mm, 223 parts, among them J201 USB_C_Receptacle_USB2.0, J202 tag-connect-swd, J5 Breakaway_Tabs, J501 tag-connect-swd, J502 USB_C_Receptacle_USB2.0, J601 tag-connect-swd, J602 USB_A, SW301 SW_Push, SW302 SW_Push, SW303 SW_Push, SW304 SW_Push, SW305 SW_Push, SW306 SW_Push, SW307 SW_Push, SW308 SW_Push, SW309 SW_Push, SW310 SW_Push, SW311 SW_Push, SW312 SW_Push, SW313 SW_Push, SW314 SW_Push, SW315 SW_Push, SW316 SW_Push, SW317 SW_Push, SW318 SW_Push, SW319 SW_Push, SW320 SW_Push, SW321 SW_Push, SW401 SW_Push, SW402 SW_Push, SW403 SW_Push, SW404 SW_Push, SW405 SW_Push, SW406 SW_Push, SW407 SW_Push, SW408 SW_Push, SW409 SW_Push, SW410 SW_Push, SW411 SW_Push, SW412 SW_Push, SW413 SW_Push, SW414 SW_Push, SW415 SW_Push, SW416 SW_Push, SW417 SW_Push, SW418 SW_Push, SW419 SW_Push, SW420 SW_Push, SW421 SW_Push, SW601 SW_Push, U201 nRF52833-QDxx, U202 USBLC6-2SC6, U204 MCP73832-2-OT, U501 nRF52833-QDxx, U502 USBLC6-2SC6, U503 MCP73832-2-OT, U601 nRF52833-QDxx, U602 USBLC6-2SC6, Y201 32 MHz, Y501 32 MHz, Y601 32 MHz

Commit message: Save
Parts:
- removed C203, C510: 4.7u, passive:C_0603
- removed D201, D501: RED, Diode_SMD:D_0603_1608Metric
- removed R205, R501: 1k, passive:R_0402
- removed REF**: Kailh Choc Hotswap 1U, connectors:Kailh Choc Hotswap 1U
- removed REF**: Hirose_FH12-10S-0.5SH_1x10-1MP_P0.50mm_Horizontal, Connector_FFC-FPC:Hirose_FH12-10S-0.5SH_1x10-1MP_P0.50mm_Horizontal
- added C217: 1u, passive:C_0402, F.Cu at (136.5, 109.5)
- added C218: 1u, passive:C_0402, F.Cu at (138.7, 109.5)
- added C224: 560p, passive:C_0402, F.Cu at (135.5, 109.5)
- added C225: 4.7u, passive:C_0603, F.Cu at (135.2, 65.0)
- added C522: 1u, passive:C_0402, F.Cu at (160.2, 41.9)
- added C523: 1u, passive:C_0402, F.Cu at (162.1, 41.9)
- added C524: 560p, passive:C_0402, F.Cu at (163.9, 41.9)
- added C525: 4.7u, passive:C_0603, F.Cu at (153.6, 29.4)
- added FB202: FerriteBead_Small, passive:R_0603, F.Cu at (137.6, 109.5)
- added FB203: FerriteBead_Small, passive:R_0603, F.Cu at (139.8, 109.5)
- added FB502: FerriteBead_Small, passive:R_0603, F.Cu at (155.8, 29.4)
- added FB503: FerriteBead_Small, passive:R_0603, F.Cu at (157.9, 29.4)
- added J203: LCD, Connector_FFC-FPC:Hirose_FH12-10S-0.5SH_1x10-1MP_P0.50mm_Horizontal, B.Cu at (137.0, 104.0)
- added J503: LCD, Connector_FFC-FPC:Hirose_FH12-10S-0.5SH_1x10-1MP_P0.50mm_Horizontal, B.Cu at (160.9, 104.0)
- added U203: TPS70630DBVR, Package_TO_SOT_SMD:SOT-23-5, F.Cu at (136.8, 67.2)
- added U504: TPS70630DBVR, Package_TO_SOT_SMD:SOT-23-5, F.Cu at (161.6, 38.0)
- moved C519 2.56 mm to (161.6, 65.0), turned to 180 degrees
- moved C219 2.52 mm to (137.7, 65.0), turned to 180 degrees
- moved C504 1.57 mm to (169.1, 62.6), turned to -90 degrees
- moved C211 1.48 mm to (145.1, 62.5), turned to -90 degrees
- moved R206 0.85 mm to (133.9, 66.7), turned to -90 degrees
Connections:
- C206 pad 1: /Left Keyboard Controller/VBAT -> /Left Keyboard Controller/VDD
- C511 pad 1: /Right Keyboard Controller/VBAT -> /Right Keyboard Controller/VDD
- SW401 pad 1: Net-(D401-A) -> /Right Keyboard Controller/KIO0
- SW401 pad 2: /Right Keyboard Controller/KIO0 -> Net-(D401-A)
- SW402 pad 1: Net-(D402-A) -> /Right Keyboard Controller/KIO1
- SW402 pad 2: /Right Keyboard Controller/KIO1 -> Net-(D402-A)
- SW403 pad 1: Net-(D403-A) -> /Right Keyboard Controller/KIO2
- SW403 pad 2: /Right Keyboard Controller/KIO2 -> Net-(D403-A)
- SW404 pad 1: Net-(D404-A) -> /Right Keyboard Controller/KIO3
- SW404 pad 2: /Right Keyboard Controller/KIO3 -> Net-(D404-A)
- SW405 pad 1: Net-(D405-A) -> /Right Keyboard Controller/KIO9
- SW405 pad 2: /Right Keyboard Controller/KIO9 -> Net-(D405-A)
- SW406 pad 1: Net-(D406-A) -> /Right Keyboard Controller/KIO8
- SW406 pad 2: /Right Keyboard Controller/KIO8 -> Net-(D406-A)
- SW407 pad 1: Net-(D407-A) -> /Right Keyboard Controller/KIO0
- SW407 pad 2: /Right Keyboard Controller/KIO0 -> Net-(D407-A)
- SW408 pad 1: Net-(D408-A) -> /Right Keyboard Controller/KIO1
- SW408 pad 2: /Right Keyboard Controller/KIO1 -> Net-(D408-A)
- SW409 pad 1: Net-(D409-A) -> /Right Keyboard Controller/KIO2
- SW409 pad 2: /Right Keyboard Controller/KIO2 -> Net-(D409-A)
- SW410 pad 1: Net-(D410-A) -> /Right Keyboard Controller/KIO3
- SW410 pad 2: /Right Keyboard Controller/KIO3 -> Net-(D410-A)
- SW411 pad 1: Net-(D411-A) -> /Right Keyboard Controller/KIO9
- SW411 pad 2: /Right Keyboard Controller/KIO9 -> Net-(D411-A)
- SW412 pad 1: Net-(D412-A) -> /Right Keyboard Controller/KIO8
- SW412 pad 2: /Right Keyboard Controller/KIO8 -> Net-(D412-A)
- SW413 pad 1: Net-(D413-A) -> /Right Keyboard Controller/KIO0
- SW413 pad 2: /Right Keyboard Controller/KIO0 -> Net-(D413-A)
- SW414 pad 1: Net-(D414-A) -> /Right Keyboard Controller/KIO1
- SW414 pad 2: /Right Keyboard Controller/KIO1 -> Net-(D414-A)
- SW415 pad 1: Net-(D415-A) -> /Right Keyboard Controller/KIO2
- SW415 pad 2: /Right Keyboard Controller/KIO2 -> Net-(D415-A)
- SW416 pad 1: Net-(D416-A) -> /Right Keyboard Controller/KIO3
- SW416 pad 2: /Right Keyboard Controller/KIO3 -> Net-(D416-A)
- SW417 pad 1: Net-(D417-A) -> /Right Keyboard Controller/KIO9
- SW417 pad 2: /Right Keyboard Controller/KIO9 -> Net-(D417-A)
- SW418 pad 1: Net-(D418-A) -> /Right Keyboard Controller/KIO8
- SW418 pad 2: /Right Keyboard Controller/KIO8 -> Net-(D418-A)
- U201 pad 2: /Left Keyboard Controller/LED -> /Left Keyboard Controller/SCLK
- U201 pad 36: unconnected-(U201-AIN7/P0.31-Pad36) -> /Left Keyboard Controller/CS
- U201 pad 6: unconnected-(U201-P1.09-Pad6) -> /Left Keyboard Controller/DATA_IN
- U201 pad 9: /Left Keyboard Controller/VBAT -> /Left Keyboard Controller/VDD
- U501 pad 2: /Right Keyboard Controller/LED -> /Right Keyboard Controller/SCLK
- U501 pad 36: unconnected-(U501-AIN7/P0.31-Pad36) -> /Right Keyboard Controller/CS
- U501 pad 6: unconnected-(U501-P1.09-Pad6) -> /Right Keyboard Controller/DATA_IN
- U501 pad 9: /Right Keyboard Controller/VBAT -> /Right Keyboard Controller/VDD
Routing:
- net /Right Keyboard Controller/KIO6: track 43.7 -> 151.9 mm
- net /Right Keyboard Controller/KIO5: track 27.5 -> 134.3 mm
- net /Right Keyboard Controller/KIO4: track 7.41 -> 112.1 mm
- net GND: track 21.8 -> 109.8 mm, vias 418 -> 415
- net /Right Keyboard Controller/KIO9: track 74.3 -> 160.4 mm, vias 1 -> 5
- net /Right Keyboard Controller/KIO3: track 75.8 -> 157.6 mm, vias 1 -> 5
- net /Right Keyboard Controller/KIO7: track 44.9 -> 119.8 mm
- net /Left Keyboard Controller/DATA_IN: track 0.00 -> 58.5 mm, vias 0 -> 3
- net /Left Keyboard Controller/CS: track 0.00 -> 56.2 mm, vias 0 -> 3
- net /Right Keyboard Controller/KIO8: track 73.0 -> 127.1 mm, vias 1 -> 5
- net /Left Keyboard Controller/SCLK: track 0.00 -> 53.8 mm, vias 0 -> 3
- net /Right Keyboard Controller/KIO1: track 86.3 -> 138.1 mm, vias 1 -> 4
- net /Right Keyboard Controller/KIO2: track 84.4 -> 133.1 mm, vias 1 -> 4
- net /Right Keyboard Controller/KIO0: track 84.1 -> 132.7 mm, vias 1 -> 4
- net /Left Keyboard Controller/VDD: track 36.1 -> 76.6 mm, vias 5 -> 7
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
Commit message: Finished routing, passing DRC
Parts:
- moved FB503 80.3 mm to (163.9, 109.5)
- moved FB502 80.3 mm to (161.7, 109.5), turned to -90 degrees
- moved C524 67.7 mm to (159.6, 109.5), turned to -90 degrees
- moved C523 67.6 mm to (162.8, 109.5)
- moved C522 67.6 mm to (160.6, 109.5)
- moved C525 36.0 mm to (159.4, 64.9), turned to 180 degrees
- moved U504 29.8 mm to (160.9, 67.8)
- moved C520 2.65 mm to (164.8, 66.9), turned to 90 degrees
- moved FB501 2.65 mm to (163.4, 66.9)
- moved R504 0.64 mm to (157.7, 64.5), turned to -90 degrees
- moved U503 0.21 mm to (165.8, 69.8)
- moved C521 0.10 mm to (166.5, 67.5)
- moved R505 0.10 mm to (158.2, 66.0)
Routing:
- net /Right Keyboard Controller/KIO0: track 132.7 -> 263.0 mm
- net /Right Keyboard Controller/KIO1: track 138.1 -> 249.4 mm
- net /Right Keyboard Controller/KIO2: track 133.1 -> 226.7 mm
- net /Right Keyboard Controller/VDD: track 37.0 -> 97.6 mm, vias 5 -> 8
- net GND: track 109.8 -> 170.2 mm, vias 415 -> 402
- net /Right Keyboard Controller/DATA_IN: track 6.77 -> 62.7 mm, vias 1 -> 3
- net /Right Keyboard Controller/SCLK: track 6.80 -> 61.5 mm, vias 1 -> 3
- net /Right Keyboard Controller/CS: track 6.66 -> 57.0 mm, vias 1 -> 3
- net /Right Keyboard Controller/KIO3: track 157.6 -> 205.2 mm
- net /Left Keyboard Controller/VDD: track 76.6 -> 103.1 mm, vias 7 -> 8
- net /Right Keyboard Controller/KIO9: track 160.4 -> 184.3 mm
- net /Right Keyboard Controller/VUSB: track 6.06 -> 19.1 mm
- net /Right Keyboard Controller/VBAT: track 8.91 -> 18.2 mm, vias 1 -> 3
- net /Right Keyboard Controller/VDDA: track 5.30 -> 10.4 mm, vias 0 -> 1
- net /Left Keyboard Controller/CS: track 56.2 -> 61.1 mm
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
Commit message: Cleanup
Routing:
- net GND: vias 402 -> 420
Other:
- board text added: "302030 Li-Ion"
- board text added: "Corne CherryBurst"
- board text added: "LS011B7DH03"
- board text removed: "502030 Li-Ion"
- board text removed: "Corne ShockBurst"
- board text removed: "TM"
