File: crkbd-shockburst.kicad_pcb (KiCad board)
At the start: 4 copper layers, 272 x 112 mm, 231 parts, among them J201 USB_C_Receptacle_USB2.0, J202 tag-connect-swd, J203 LCD, J5 Breakaway_Tabs, J501 tag-connect-swd, J502 USB_C_Receptacle_USB2.0, J503 LCD, J601 tag-connect-swd, J602 USB_A, SW301 SW_Push, SW302 SW_Push, SW303 SW_Push, SW304 SW_Push, SW305 SW_Push, SW306 SW_Push, SW307 SW_Push, SW308 SW_Push, SW309 SW_Push, SW310 SW_Push, SW311 SW_Push, SW312 SW_Push, SW313 SW_Push, SW314 SW_Push, SW315 SW_Push, SW316 SW_Push, SW317 SW_Push, SW318 SW_Push, SW319 SW_Push, SW320 SW_Push, SW321 SW_Push, SW401 SW_Push, SW402 SW_Push, SW403 SW_Push, SW404 SW_Push, SW405 SW_Push, SW406 SW_Push, SW407 SW_Push, SW408 SW_Push, SW409 SW_Push, SW410 SW_Push, SW411 SW_Push, SW412 SW_Push, SW413 SW_Push, SW414 SW_Push, SW415 SW_Push, SW416 SW_Push, SW417 SW_Push, SW418 SW_Push, SW419 SW_Push, SW420 SW_Push, SW421 SW_Push, SW601 SW_Push, U201 nRF52833-QDxx, U202 USBLC6-2SC6, U203 TPS70630DBVR, U204 MCP73832-2-OT, U501 nRF52833-QDxx, U502 USBLC6-2SC6, U503 MCP73832-2-OT, U504 TPS70630DBVR, U601 nRF52833-QDxx, U602 USBLC6-2SC6, Y201 32 MHz, Y501 32 MHz, Y601 32 MHz

Commit message: Add power switch
Parts:
- added SW101: SW_SPDT, connectors:SSSS810701, F.Cu at (145.5, 111.8)
- added SW102: SW_SPDT, connectors:SSSS810701, F.Cu at (152.2, 111.8)
Connections:
- U203 pad 3: /Left Keyboard Controller/VBAT -> /Left Keyboard Controller/POWER_EN
- U504 pad 3: /Right Keyboard Controller/VBAT -> /Right Keyboard Controller/POWER_EN
Routing:
- net GND: track 170.2 -> 236.1 mm, vias 420 -> 422
- net /Left Keyboard Controller/POWER_EN: track 0.00 -> 50.2 mm, vias 0 -> 2
- net /Right Keyboard Controller/POWER_EN: track 0.00 -> 50.0 mm, vias 0 -> 2
- net /Left Keyboard Controller/VBAT: track 18.3 -> 16.9 mm
- net /Right Keyboard Controller/VBAT: track 18.2 -> 17.0 mm, vias 3 -> 2
Other:
- board text added: "OFF"
- board text added: "POWER OFF"
