File: crkbd-shockburst.kicad_sch (KiCad schematic)
At the start: 0 parts

Commit message: Schematics
Parts:
- added Ant201: antenna, RF_Antenna:Texas_SWRA117D_2.4GHz_Right, symbol antennas:antenna
Connections:
- new net GND: Ant201.2
- new net Left Keyboard Half/ANT: Ant201.1
Other:
- added sheet Left Keyboard Half (keyboard_half.kicad_sch)
Changed lines of the file:
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@@
 (kicad_sch (version 20230121) (generator eeschema)
   (paper "A4")
+  (wire (pts (xy 52.07 80.01) (xy 57.15 80.01))
+    (stroke (width 0) (type default))
+  )
+  (symbol (lib_id "power:GND") (at 52.07 77.47 90) (unit 1)
+    (in_bom yes) (on_board yes) (dnp no) (fields_autoplaced)
+    (property "Reference" "#PWR0237" (at 58.42 77.47 0)
+      (effects (font (size 1.27 1.27)) hide)
+    )
+    (property "Value" "GND" (at 57.15 77.47 0)
+      (effects (font (size 1.27 1.27)) hide)
+    )
+    (property "Footprint" "" (at 52.07 77.47 0)
+      (effects (font (size 1.27 1.27)) hide)
+    )
+    (property "Datasheet" "" (at 52.07 77.47 0)
+      (effects (font (size 1.27 1.27)) hide)
+    )
+    (pin "1")
+    (instances
+      (project "crkbd-shockburst"
+        (path "/76f7b6ad-1528-4ee8-9fc0-4578616aebf5/03cbda14-d368-4dde-b0d5-76768308216d"
+          (reference "#PWR0237") (unit 1)
+        )
+        (path "/76f7b6ad-1528-4ee8-9fc0-4578616aebf5"
+          (reference "#PWR0101") (unit 1)
+        )
+      )
+    )
+  )
+  (symbol (lib_id "antennas:antenna") (at 46.99 80.01 0) (unit 1)
+    (in_bom no) (on_board yes) (dnp no) (fields_autoplaced)
+    (property "Reference" "Ant201" (at 46.99 71.12 0)
+      (effects (font (size 1.27 1.27)))
+    )
+    (property "Value" "antenna" (at 46.99 82.55 0)
+      (effects (font (size 1.27 1.27)) hide)
+    )
+    (property "Footprint" "RF_Antenna:Texas_SWRA117D_2.4GHz_Right" (at 46.99 80.01 0)
+      (effects (font (size 1.27 1.27)) hide)
+    )
+    (property "Datasheet" "" (at 46.99 72.39 0)
+      (effects (font (size 1.27 1.27)))
+    )
+    (property "MFPN" "" (at 46.99 80.01 0)
+      (effects (font (size 1.27 1.27)) hide)
+    )
+    (property "Specification" "" (at 46.99 80.01 0)
+      (effects (font (size 1.27 1.27)) hide)
+    )
+    (property "LCSC" "" (at 46.99 80.01 0)
+      (effects (font (size 1.27 1.27)) hide)
+    )
+    (pin "1")
+    (pin "2")
+    (instances
+      (project "crkbd-shockburst"
+        (path "/76f7b6ad-1528-4ee8-9fc0-4578616aebf5/03cbda14-d368-4dde-b0d5-76768308216d"
+          (reference "Ant201") (unit 1)
+        )
+        (path "/76f7b6ad-1528-4ee8-9fc0-4578616aebf5"
+          (reference "Ant101") (unit 1)
+        )
+      )
+    )
+  )
+  (sheet (at 57.15 73.66) (size 27.94 11.43) (fields_autoplaced)
+    (stroke (width 0.1524) (type solid))
+    (fill (color 0 0 0 0.0000))
+    (property "Sheetname" "Left Keyboard Half" (at 57.15 72.9484 0)
+      (effects (font (size 1.27 1.27)) (justify left bottom))
+    )
+    (property "Sheetfile" "keyboard_half.kicad_sch" (at 57.15 85.6746 0)
+      (effects (font (size 1.27 1.27)) (justify left top))
+    )
+    (pin "ANT" input (at 57.15 80.01 180)
+      (effects (font (size 1.27 1.27)) (justify left))
+    )
+    (instances
+      (project "crkbd-shockburst"
+        (path "/76f7b6ad-1528-4ee8-9fc0-4578616aebf5" (page "2"))
+      )
+    )
+  )
   (sheet_instances
     (path "/" (page "1"))

Commit message: Layout
Parts:
- added Ant201: antenna, RF_Antenna:Texas_SWRA117D_2.4GHz_Right, symbol antennas:antenna
- added R205: 1k, passive:R_0402, symbol Device:R_Small
Connections:
- net GND: now also Ant201.2, R205.1
- new net Left Keyboard Controller/LEFT: R205.2
- new net Right Keyboard Controller/ANT: Ant201.1
- no-connect marks 0 -> 1
Other:
- sheet Left Keyboard Half renamed Left Keyboard Controller
- added sheet Left switches (left_switches.kicad_sch)
- added sheet Right Keyboard Controller (keyboard_half.kicad_sch)
- added sheet Right Switches (right_switches.kicad_sch)
- added sheet USB Dongle (usb_dongle.kicad_sch)
- sheet Left Keyboard Controller ports: added KIO0, KIO1, KIO2, KIO3, KIO4, KIO5, KIO6, KIO7, KIO8, KIO9, LEFT; removed none

Commit message: Add power switch
Parts:
- added SW501 (x2): SW_SPDT, connectors:SSSS810701, symbol Switch:SW_SPDT
Connections:
- net GND: now also SW501.2 (B), SW501.2 (B)
- new net Left Keyboard Controller/POWER_EN: SW501.1 (A)
- new net Right Keyboard Controller/POWER_EN: SW501.3 (C)
- no-connect marks 1 -> 3
Other:
- sheet Left Keyboard Controller ports: added POWER_EN; removed none
- sheet Right Keyboard Controller ports: added POWER_EN; removed none
Changed lines of the file:
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@@
 (kicad_sch (version 20230121) (generator eeschema)
   (paper "A4")
+  (no_connect (at 35.56 92.71))
   (no_connect (at 57.15 138.43))
+  (no_connect (at 35.56 125.73))
   (wire (pts (xy 85.09 99.06) (xy 121.92 99.06))
     (stroke (width 0) (type default))
@@
     (stroke (width 0) (type default))
   )
+  (wire (pts (xy 35.56 130.81) (xy 57.15 130.81))
+    (stroke (width 0) (type default))
+  )
   (wire (pts (xy 53.34 96.52) (xy 57.15 96.52))
     (stroke (width 0) (type default))
@@
   )
   (wire (pts (xy 85.09 135.89) (xy 104.14 135.89))
+    (stroke (width 0) (type default))
+  )
+  (wire (pts (xy 35.56 87.63) (xy 57.15 87.63))
     (stroke (width 0) (type default))
   )
@@
     )
   )
+  (symbol (lib_id "power:GND") (at 25.4 128.27 270) (unit 1)
+    (in_bom yes) (on_board yes) (dnp no) (fields_autoplaced)
+    (property "Reference" "#PWR0214" (at 19.05 128.27 0)
+      (effects (font (size 1.27 1.27)) hide)
+    )
+    (property "Value" "GND" (at 20.32 128.27 0)
+      (effects (font (size 1.27 1.27)) hide)
+    )
+    (property "Footprint" "" (at 25.4 128.27 0)
+      (effects (font (size 1.27 1.27)) hide)
+    )
+    (property "Datasheet" "" (at 25.4 128.27 0)
+      (effects (font (size 1.27 1.27)) hide)
+    )
+    (pin "1")
+    (instances
+      (project "crkbd-shockburst"
+        (path "/76f7b6ad-1528-4ee8-9fc0-4578616aebf5/03cbda14-d368-4dde-b0d5-76768308216d"
+          (reference "#PWR0214") (unit 1)
+        )
+        (path "/76f7b6ad-1528-4ee8-9fc0-4578616aebf5/3b44a955-2a37-4d30-8a82-5f0155f54e66"
+          (reference "#PWR0510") (unit 1)
+        )
+        (path "/76f7b6ad-1528-4ee8-9fc0-4578616aebf5"
+          (reference "#PWR0106") (unit 1)
+        )
+      )
+    )
+  )
   (symbol (lib_id "power:GND") (at 52.07 77.47 90) (unit 1)
     (in_bom yes) (on_board yes) (dnp no) (fields_autoplaced)
@@
     )
   )
+  (symbol (lib_id "power:GND") (at 25.4 90.17 270) (unit 1)
+    (in_bom yes) (on_board yes) (dnp no) (fields_autoplaced)
+    (property "Reference" "#PWR0214" (at 19.05 90.17 0)
+      (effects (font (size 1.27 1.27)) hide)
+    )
+    (property "Value" "GND" (at 20.32 90.17 0)
+      (effects (font (size 1.27 1.27)) hide)
+    )
+    (property "Footprint" "" (at 25.4 90.17 0)
+      (effects (font (size 1.27 1.27)) hide)
+    )
+    (property "Datasheet" "" (at 25.4 90.17 0)
+      (effects (font (size 1.27 1.27)) hide)
+    )
+    (pin "1")
+    (instances
+      (project "crkbd-shockburst"
+        (path "/76f7b6ad-1528-4ee8-9fc0-4578616aebf5/03cbda14-d368-4dde-b0d5-76768308216d"
+          (reference "#PWR0214") (unit 1)
+        )
+        (path "/76f7b6ad-1528-4ee8-9fc0-4578616aebf5/3b44a955-2a37-4d30-8a82-5f0155f54e66"
+          (reference "#PWR0510") (unit 1)
+        )
+        (path "/76f7b6ad-1528-4ee8-9fc0-4578616aebf5"
+          (reference "#PWR0105") (unit 1)
+        )
+      )
+    )
+  )
+  (symbol (lib_id "Switch:SW_SPDT") (at 30.48 90.17 0) (unit 1)
+    (in_bom yes) (on_board yes) (dnp no) (fields_autoplaced)
+    (property "Reference" "SW501" (at 30.48 82.55 0)
+      (effects (font (size 1.27 1.27)))
+    )
+    (property "Value" "SW_SPDT" (at 30.48 85.09 0)
+      (effects (font (size 1.27 1.27)))
+    )
+    (property "Footprint" "connectors:SSSS810701" (at 30.48 90.17 0)
+      (effects (font (size 1.27 1.27)) hide)
+    )
+    (property "Datasheet" "~" (at 30.48 90.17 0)
+      (effects (font (size 1.27 1.27)) hide)
+    )
+    (property "MFPN" "SSSS810701" (at 30.48 90.17 0)
+      (effects (font (size 1.27 1.27)) hide)
+    )
+    (property "Specification" "" (at 30.48 90.17 0)
+      (effects (font (size 1.27 1.27)) hide)
+    )
+    (property "LCSC" "C97433" (at 30.48 90.17 0)
+      (effects (font (size 1.27 1.27)) hide)
+    )
+    (pin "1")
+    (pin "2")
+    (pin "3")
+    (instances
+      (project "crkbd-shockburst"
+        (path "/76f7b6ad-1528-4ee8-9fc0-4578616aebf5/3b44a955-2a37-4d30-8a82-5f0155f54e66"
+          (reference "SW501") (unit 1)
+        )
+        (path "/76f7b6ad-1528-4ee8-9fc0-4578616aebf5/03cbda14-d368-4dde-b0d5-76768308216d"
+          (reference "SW201") (unit 1)
+        )
+        (path "/76f7b6ad-1528-4ee8-9fc0-4578616aebf5"
+          (reference "SW101") (unit 1)
+        )
+      )
+    )
+  )
   (symbol (lib_id "Device:R_Small") (at 50.8 96.52 90) (unit 1)
     (in_bom yes) (on_board yes) (dnp no) (fields_autoplaced)
@@
         (path "/76f7b6ad-1528-4ee8-9fc0-4578616aebf5"
           (reference "R101") (unit 1)
+        )
+      )
+    )
+  )
+  (symbol (lib_id "Switch:SW_SPDT") (at 30.48 128.27 0) (unit 1)
+    (in_bom yes) (on_board yes) (dnp no) (fields_autoplaced)
+    (property "Reference" "SW501" (at 30.48 120.65 0)
+      (effects (font (size 1.27 1.27)))
+    )
+    (property "Value" "SW_SPDT" (at 30.48 123.19 0)
+      (effects (font (size 1.27 1.27)))
+    )
+    (property "Footprint" "connectors:SSSS810701" (at 30.48 128.27 0)
+      (effects (font (size 1.27 1.27)) hide)
+    )
+    (property "Datasheet" "~" (at 30.48 128.27 0)
+      (effects (font (size 1.27 1.27)) hide)
+    )
+    (property "MFPN" "SSSS810701" (at 30.48 128.27 0)
+      (effects (font (size 1.27 1.27)) hide)
+    )
+    (property "Specification" "" (at 30.48 128.27 0)
+      (effects (font (size 1.27 1.27)) hide)
+    )
+    (property "LCSC" "C97433" (at 30.48 128.27 0)
+      (effects (font (size 1.27 1.27)) hide)
+    )
+    (pin "1")
+    (pin "2")
+    (pin "3")
+    (instances
+      (project "crkbd-shockburst"
+        (path "/76f7b6ad-1528-4ee8-9fc0-4578616aebf5/3b44a955-2a37-4d30-8a82-5f0155f54e66"
+          (reference "SW501") (unit 1)
+        )
+        (path "/76f7b6ad-1528-4ee8-9fc0-4578616aebf5/03cbda14-d368-4dde-b0d5-76768308216d"
+          (reference "SW201") (unit 1)
+        )
+        (path "/76f7b6ad-1528-4ee8-9fc0-4578616aebf5"
+          (reference "SW102") (unit 1)
         )
       )
@@
       (effects (font (size 1.27 1.27)) (justify left))
     )
+    (pin "POWER_EN" input (at 57.15 87.63 180)
+      (effects (font (size 1.27 1.27)) (justify left))
+    )
     (instances
       (project "crkbd-shockburst"
@@
       (effects (font (size 1.27 1.27)) (justify left))
     )
+    (pin "POWER_EN" input (at 57.15 130.81 180)
+      (effects (font (size 1.27 1.27)) (justify left))
+    )
