File: keyboard_half.kicad_sch (KiCad schematic)
At the start: 86 parts, among them J201 USB_C_Receptacle_USB2.0, J202 tag-connect-swd, SW201 SW_Push, SW202 SW_Push, SW203 SW_Push, SW204 SW_Push, SW205 SW_Push, SW206 SW_Push, SW207 SW_Push, SW208 SW_Push, SW209 SW_Push, SW210 SW_Push, SW211 SW_Push, SW212 SW_Push, SW213 SW_Push, SW214 SW_Push, SW215 SW_Push, SW216 SW_Push, SW217 SW_Push, SW218 SW_Push, SW219 SW_Push, SW220 SW_Push, SW221 SW_Push, U201 nRF52833-QDxx, U202 USBLC6-2SC6, U204 MCP73832-2-OT, Y201 32 MHz, Y202 32 kHz

Commit message: Layout
Parts:
- removed C217, C218: 10p, passive:C_0402, symbol Device:C_Small
- removed D201, D202, D203, D204, D205, D206, D207, D208, D209, D210, D211, D212, D213, D214, D215, D216, D217, D218, D219, D220, D221: 1N4148W, Diode_SMD:D_SOD-123, symbol Device:D_Small
- removed SW201, SW202, SW203, SW204, SW205, SW206, SW207, SW208, SW209, SW210, SW211, SW212, SW213, SW214, SW215, SW216, SW217, SW218, SW219, SW220, SW221: SW_Push, connectors:Kailh MX hotswap socket, symbol Switch:SW_Push
- removed Y202: 32 kHz, Crystal:Crystal_SMD_3215-2Pin_3.2x1.5mm, symbol Device:Crystal_Small
- added H201, H202, H203, H204, H205: MountingHole, MountingHole:MountingHole_4.3mm_M4, symbol Mechanical:MountingHole
- BT201: footprint (none) -> connectors:1x2_2.54mm
- D201: renamed from D222; footprint Diode_SMD:D_0805_2012Metric -> Diode_SMD:D_0603_1608Metric; LCSC C5160694 -> C497930; MFPN A-SP170R6C-A01-3T -> HL-PST-1608S9AC-CZ
- J202: footprint connectors:tag-connect_6pin_nolegs_swd -> Connector:Tag-Connect_TC2030-IDC-NL_2x03_P1.27mm_Vertical; now left out of the parts list
Connections:
- net COL4 is gone; now on net CHG_STAT: U201.17 (P0.20)
- net XL1 is gone; now on net LED: U201.2 (XL1/P0.00)
- net CHG_STAT: no longer U201.4 (AIN2/P0.04)
- net LED: no longer U201.5 (AIN3/P0.05)
- net VBAT_MEAS: now also U201.31 (AIN1/P0.03); no longer U201.32 (AIN0/P0.02)
- net LEFT: now reaches U201.22 (NFC1/P0.09)
- net +BATT renamed VBAT
- net COL0 renamed KIO0
- net COL1: no longer names the net of U201.7 (P0.11)
- net COL2 renamed KIO2
- net COL3 renamed KIO1
- net COL5 renamed KIO9
- net RESET: no longer names the net of U201.16 (P0.18/~{RESET})
- net RESET: no longer J202.3 (~{RESET})
- net ROW0 renamed KIO8
- net ROW1 renamed KIO7
- net ROW2: no longer names the net of U201.36 (AIN7/P0.31)
- net ROW3: no longer names the net of U201.6 (P1.09)
- net VBUS renamed VUSB
- net XL2 renamed KIO6
- new net KIO3: U201.32 (AIN0/P0.02)
- new net KIO4: U201.5 (AIN3/P0.05)
- new net KIO5: U201.4 (AIN2/P0.04)
- no-connect marks 5 -> 8
Other:
- moved on the sheet: C203, C204, C205, C206, C207, C208, C209, C210, C211, C212, C213, C214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

Commit message: Save
Parts:
- removed C203: 4.7u, passive:C_0603, symbol Device:C_Small
- removed D201: RED, Diode_SMD:D_0603_1608Metric, symbol Device:LED_Small
- removed R205: 1k, passive:R_0402, symbol Device:R_Small
- added C217, C218: 1u, passive:C_0402, symbol Device:C_Small
- added C224: 560p, passive:C_0402, symbol Device:C_Small
- added C225: 4.7u, passive:C_0603, symbol Device:C_Small
- added FB202, FB203: FerriteBead_Small, passive:R_0603, symbol Device:FerriteBead_Small
- added J203: LCD, Connector_FFC-FPC:Hirose_FH12-10S-0.5SH_1x10-1MP_P0.50mm_Horizontal, symbol Connector_Generic_MountingPin:Conn_01x10_MountingPin
- added U203: TPS70630DBVR, Package_TO_SOT_SMD:SOT-23-5, symbol Regulator_Linear:TPS7A0533PDBV
Connections:
- net GND: now also C217.1, C218.1, C224.2, C225.2, FB203.1, J203.4 (Pin_4), J203.8 (Pin_8), J203.9 (Pin_9), J203.MP (MountPin), U203.2 (GND)
- net VBAT: now also U203.1 (IN), U203.3 (EN); no longer C206.1, U201.9 (VDDH)
- net VDD: now also C206.1, U201.9 (VDDH), C218.2, C225.1, FB202.1, J203.7 (Pin_7), U203.5 (OUT)
- net CS: now reaches U201.36 (AIN7/P0.31)
- net CS: now also J203.3 (Pin_3)
- net DATA_IN: now reaches U201.6 (P1.09)
- net DATA_IN: now also J203.2 (Pin_2)
- net LED renamed SCLK
- net SCLK: now also J203.1 (Pin_1)
- new net DISP: C224.1, J203.5 (Pin_5)
- new net VDDA: C217.2, FB202.2, J203.6 (Pin_6)
- new net VSSA: FB203.2, J203.10 (Pin_10)
- no-connect marks 8 -> 6
Other:
- note removed: "Battery Status LED"
- moved on the sheet: C206, H201, H202, H203, H204, H205

Commit message: Add power switch
Connections:
- net VBAT: no longer U203.3 (EN)
- new net POWER_EN: U203.3 (EN)
Changed lines of the file:
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@@
   (junction (at 157.48 64.77) (diameter 0) (color 0 0 0 0)
-  )
-  (junction (at 43.18 118.11) (diameter 0) (color 0 0 0 0)
   )
   (junction (at 69.85 118.11) (diameter 0) (color 0 0 0 0)
@@
     (stroke (width 0) (type default))
   )
-  (wire (pts (xy 43.18 120.65) (xy 43.18 118.11))
-    (stroke (width 0) (type default))
-  )
   (wire (pts (xy 50.8 151.13) (xy 73.66 151.13))
     (stroke (width 0) (type default))
@@
     (stroke (width 0) (type default))
   )
-  (wire (pts (xy 45.72 120.65) (xy 43.18 120.65))
+  (wire (pts (xy 45.72 120.65) (xy 31.75 120.65))
     (stroke (width 0) (type default))
   )
@@
     (stroke (width 0) (type default))
   )
-  (wire (pts (xy 43.18 118.11) (xy 45.72 118.11))
+  (wire (pts (xy 31.75 118.11) (xy 45.72 118.11))
     (stroke (width 0) (type default))
   )
@@
     (stroke (width 0) (type default))
   )
-  (wire (pts (xy 31.75 118.11) (xy 43.18 118.11))
-    (stroke (width 0) (type default))
-  )
   (text "200 mA charging" (at 97.79 193.04 0)
     (effects (font (size 1.27 1.27)) (justify left bottom))
@@
     (effects (font (size 1.27 1.27)) (justify left))
   )
+  (hierarchical_label "POWER_EN" (shape input) (at 31.75 120.65 180) (fields_autoplaced)
+    (effects (font (size 1.27 1.27)) (justify right))
+  )
   (hierarchical_label "LEFT" (shape bidirectional) (at 190.5 86.36 0) (fields_autoplaced)
