File: chocburst/crkbd-shockburst.kicad_pcb (KiCad board)
At the start: 4 copper layers, 272 x 112 mm, 233 parts, among them J201 USB_C_Receptacle_USB2.0, J202 tag-connect-swd, J203 LCD, J204 Conn_01x02_MountingPin, J5 Breakaway_Tabs, J501 tag-connect-swd, J502 USB_C_Receptacle_USB2.0, J503 LCD, J504 Conn_01x02_MountingPin, J601 tag-connect-swd, J602 USB_A, SW101 SW_SPDT, SW102 SW_SPDT, SW301 SW_Push, SW302 SW_Push, SW303 SW_Push, SW304 SW_Push, SW305 SW_Push, SW306 SW_Push, SW307 SW_Push, SW308 SW_Push, SW309 SW_Push, SW310 SW_Push, SW311 SW_Push, SW312 SW_Push, SW313 SW_Push, SW314 SW_Push, SW315 SW_Push, SW316 SW_Push, SW317 SW_Push, SW318 SW_Push, SW319 SW_Push, SW320 SW_Push, SW321 SW_Push, SW401 SW_Push, SW402 SW_Push, SW403 SW_Push, SW404 SW_Push, SW405 SW_Push, SW406 SW_Push, SW407 SW_Push, SW408 SW_Push, SW409 SW_Push, SW410 SW_Push, SW411 SW_Push, SW412 SW_Push, SW413 SW_Push, SW414 SW_Push, SW415 SW_Push, SW416 SW_Push, SW417 SW_Push, SW418 SW_Push, SW419 SW_Push, SW420 SW_Push, SW421 SW_Push, SW601 SW_Push, U201 nRF52833-QDxx, U202 USBLC6-2SC6, U203 TPS70630DBVR, U204 MCP73832-2-OT, U501 nRF52833-QDxx, U502 USBLC6-2SC6, U503 MCP73832-2-OT, U504 TPS70630DBVR, U601 nRF52833-QDxx, U602 USBLC6-2SC6, Y201 32 MHz, Y501 32 MHz, Y601 32 MHz

Commit message: Add Chocolate switch version
Parts:
- R206, R506: value 5.1k -> 10k
- SW301, SW302, SW303, SW304, SW305, SW306, SW307, SW308, SW309, SW310, SW311, SW312, SW313, SW314, SW315, SW316, SW317, SW318, SW319, SW320, SW401, SW402, SW403, SW404, SW405, SW406, SW407, SW408, SW409, SW410, SW411, SW412, SW413, SW414, SW415, SW416, SW417, SW418, SW419, SW420: footprint connectors:Kailh MX hotswap socket -> connectors:Kailh Choc Hotswap 1U
- SW321, SW421: footprint connectors:Kailh MX hotswap socket 1.5u -> connectors:Kailh Choc Hotswap 1.5U
- moved D419 3.54 mm to (218.0, 117.0), turned to -90 degrees
- moved D420 3.54 mm to (196.5, 117.5), turned to -90 degrees
- turned D301 to -90 degrees
- turned D302 to -90 degrees
- turned D303 to -90 degrees
- turned D304 to -90 degrees
- turned D305 to -90 degrees
- turned D306 to -90 degrees
- turned D307 to -90 degrees
- turned D308 to -90 degrees
- turned D309 to -90 degrees
- turned D310 to -90 degrees
- turned D311 to -90 degrees
- turned D312 to -90 degrees
- turned D313 to -90 degrees
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Routing:
- net /Left Keyboard Controller/KIO6: track 212.2 -> 194.0 mm
- net /Left Keyboard Controller/KIO8: track 175.7 -> 158.0 mm
- net /Right Keyboard Controller/KIO7: track 124.2 -> 141.2 mm
- net /Left Keyboard Controller/KIO7: track 196.5 -> 180.7 mm
- net /Right Keyboard Controller/KIO9: track 184.3 -> 170.6 mm
- net /Right Keyboard Controller/KIO3: track 205.2 -> 191.9 mm
- net Net-(D321-A): track 4.19 -> 16.2 mm
- net /Right Keyboard Controller/KIO0: track 263.0 -> 251.8 mm
- net /Left Keyboard Controller/KIO2: track 175.7 -> 164.5 mm
- net /Right Keyboard Controller/KIO2: track 226.7 -> 216.5 mm
- net /Right Keyboard Controller/KIO1: track 249.4 -> 239.2 mm
- net /Left Keyboard Controller/KIO5: track 225.0 -> 215.4 mm
- net /Right Keyboard Controller/KIO8: track 127.3 -> 136.6 mm, vias 5 -> 4
- net /Left Keyboard Controller/KIO3: track 119.9 -> 113.1 mm
- net /Left Keyboard Controller/VBAT: track 14.6 -> 20.3 mm
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Other:
- board text added: "Chg = 100 mA"
- board text added: "Corne ChocBurst"
- board text removed: "Chg = 200 mA"
- board text removed: "Corne CherryBurst"
- board text removed: "POWER OFF"
