File: top-plate/top-plate.kicad_pcb (KiCad board)
At the start: 2 copper layers, 134 x 92.8 mm, 26 parts, among them SW2 KEY_SWITCH

Commit message: Update top plate
Other:
- outline, holes or cut-outs redrawn
- board text removed: "Corne ShockBurst"
